File: Metro THM+LDO Rev C - CP2104.sch (EAGLE design)
At the start: 60 parts, among them T1 DMP3098L, T2 DMP3098L, U1 NCP1117ST50T3G, U3 CP2104, U4 AP2112-3.3, U5 LMV358IDGKR, X3 20329, Y2 CSTCE16M0V53-R0 16MHZ

Commit message: Readability Improvements to Metro RevC Schematic
Moved CP2104 from off-page into USB/Serial section of schematic.
Changed Reset Level Shifting note to correctly refer to the CP2104 instead of the old FTDI chip.
Moved some things arround slightly to reduce text overlaps.
Adjusted net routing around CP2104 to improve clarity.
Added PDF Export for Metro Rev C Schematic.
Other:
- note added: "The CP2104 chip outputs 3.3V logic, but with CMOS logic this is right at the limit of logic high on a 5V device (5V*0.7=3.5V). If the temperature rises, the required transition level will increase and may fail in some situations."
- note removed: "The FTDI chip outputs 3.3V logic, but with CMOS logic this is right at the limit of logic high on a 5V device (5V*0.7=3.5V). If the temperature rises, the required transition level will increase and may fail in some situations."
- moved on the sheet: C13, C3, C7, C9, D1, F2, FB2, GROUND1, JP1, R1, R3, R7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
